Commit message: added everything thorugh first xacro file

File: newrobot.urdf (robot description, URDF)
Before this commit: robot robot, 6 links, 5 joints
Joints:
- removed joint base_wheel_left
- added joint base_wheel_left_joint: type fixed, parent base, child wheel_left, origin xyz=-0.1 0.4 0, limit effort=1 velocity=1

File: urdf/robot.urdf (robot description, URDF)
Before this commit: robot robot, 6 links, 5 joints
Joints:
- removed joint base_wheel_left
- added joint base_wheel_left_joint: type fixed, parent base, child wheel_left, origin xyz=-0.1 0.4 0, limit effort=1 velocity=1

File: urdf/torobot.xacro (robot description, xacro)
@@ -1,4 +1,4 @@
 <?xml version="1.0"?>
-<robot name="robot">
+<robot xmlns:xacro="http://www.ros.org/wiki/xacro" name="robot">
   <link name="base">
     <visual>
@@ -64,5 +64,6 @@
     </collision>
   </link>
-  <link name="wheel_left">
+  <xacro:macro name="xacro_name" params="suffix reflect">
+  <link name="wheel_${suffix}">
     <visual>
       <geometry>
@@ -78,4 +79,12 @@
     </collision>
   </link>
+  <joint name="base_wheel_${suffix}_joint" type="fixed">
+	<parent link="base"/>
+	<child link="wheel_${suffix}"/>
+	<origin xyz="-0.1 0.4 0"/>
+	<limit velocity = "1" effort = "1"/>
+  </joint>
+  </xacro:macro>
+  <xacro:xacro_name suffix="left" reflect="1" />
   <joint name="base_laser_vert_bottom_joint" type="fixed">
     <parent link="base"/>
@@ -98,9 +107,3 @@
     <origin xyz="0.2325 0.0001 1.9201"/>
   </joint>
-  <joint name="base_wheel_left" type="fixed">
-	<parent link="base"/>
-	<child link="wheel_left"/>
-	<origin xyz="-0.1 0.4 0"/>
-	<limit velocity = "1" effort = "1"/>
-  </joint>
 </robot>
