Commit message: all work done, wheel axes need fixing

File: urdf/newrobot.urdf (robot description, URDF)
Before this commit: robot robot, 6 links, 5 joints
Links:
- added link laser_horiz_base_link, mass 0.83; collision cylinder length=0.0717 radius=0.0516; visual mesh filename=package://velodyne_description/meshes/VLP16_base_1.dae
- added link wheel_center; collision cylinder length=0.05 radius=0.15; visual cylinder length=0.05 radius=0.15
- added link wheel_right; collision cylinder length=0.05 radius=0.2; visual cylinder length=0.05 radius=0.2
- link laser_horiz: mass None -> 0.01; geometry visual mesh filename=package://velodyne_description/meshes/VLP16_scan.dae
- link laser_vert_bottom: mass None -> 1e-5; geometry collision box size=0.1 0.1 0.1; visual mesh filename=package://gazebo_plugins/test/multi_robot_scenario/meshes/l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
- link laser_vert_top_left: mass None -> 1e-5; geometry collision box size=0.1 0.1 0.1; visual mesh filename=package://gazebo_plugins/test/multi_robot_scenario/meshes/l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
- link laser_vert_top_right: mass None -> 1e-5; geometry collision box size=0.1 0.1 0.1; visual mesh filename=package://gazebo_plugins/test/multi_robot_scenario/meshes/l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
Joints:
- removed joint base_laser_horiz_joint
- added joint base_wheel_center_joint: type continuous, parent base, child wheel_center, origin xyz=0.1 0.0 -0.025 rpy=-1.57079 0 0, limit effort=1 velocity=1
- added joint base_wheel_right_joint: type continuous, parent base, child wheel_right, origin xyz=-0.1 -0.4 -0.0 rpy=-1.57079 0 0, limit effort=1 velocity=1
- added joint laser_horiz_base_mount_joint: type fixed, parent base, child laser_horiz_base_link, origin xyz=0.2325416305773505 -0.0001380069427607134 1.920122926231907 rpy=-0.0012068 0.114646 -0.0015308
- added joint laser_horiz_base_scan_joint: type fixed, parent laser_horiz_base_link, child laser_horiz, origin xyz=0 0 0.0377 rpy=0 0 0
- joint base_laser_vert_bottom_joint: axis (none) -> 0 0 1; origin xyz=0.3158 -0.0021 0.5100 -> xyz=0.3157894464801903 -0.002068548615034871 0.5099999434059285 rpy=3.1354753 -1.3045001 0.0024658
- joint base_laser_vert_top_left_joint: axis (none) -> 0 0 1; origin xyz=0.2997 0.1531 1.8443 -> xyz=0.2997 0.1531 1.8443 rpy=1.1780 0.6198 0.087
- joint base_laser_vert_top_right_joint: axis (none) -> 0 0 1; origin xyz=0.2978 -0.1450 1.8451 -> xyz=0.2978 -0.1450 1.8451 rpy=-1.1760 0.6313 -1.9377
- joint base_wheel_left_joint: origin xyz=-0.1 0.4 0 -> xyz=-0.1 0.4 -0.0 rpy=-1.57079 0 0; type fixed -> continuous

File: urdf/torobot.xacro (robot description, xacro)
@@ -14,96 +14,41 @@
     </collision>
   </link>
-  <link name="laser_vert_bottom">
+	<!-- Include the XACRO file that defines a Hokuyo LIDAR. -->
+	<xacro:include filename="$(find gazebo_plugins)/test/multi_robot_scenario/xacro/laser/hokuyo.xacro" />
+	<xacro:laser name="laser_vert_bottom" parent="base" xyz="0.3157894464801903 -0.002068548615034871 0.5099999434059285" rpy="3.1354753 -1.3045001 0.0024658" meshes="package://gazebo_plugins/test/multi_robot_scenario/meshes/laser" />
+	<xacro:laser name="laser_vert_top_left" parent="base" xyz="0.2997 0.1531 1.8443" rpy="1.1780 0.6198 0.087" meshes="package://gazebo_plugins/test/multi_robot_scenario/meshes/laser" />
+	<xacro:laser name="laser_vert_top_right" parent="base" xyz="0.2978 -0.1450 1.8451" rpy="-1.1760 0.6313 -1.9377" meshes="package://gazebo_plugins/test/multi_robot_scenario/meshes/laser" />
+	<!-- Include the XACRO file that defines a Hokuyo LIDAR. -->
+	<xacro:include filename="$(find velodyne_description)/urdf/VLP-16.urdf.xacro"/>
+	<!-- Invoke the macro to define the Hokuyo LIDAR. -->
+	<VLP-16 parent="base" name="laser_horiz" topic="laser_horiz/packets" hz="10"
+	samples="440" gpu="false">
+	<origin xyz="0.2325416305773505 -0.0001380069427607134 1.920122926231907"
+	rpy="-0.0012068 0.114646 -0.0015308" />
+	</VLP-16>
+  <xacro:macro name="xacro_name" params="suffix reflect center">
+  <link name="wheel_${suffix}">
     <visual>
       <geometry>
-        <box size="0.062 0.062 0.087"/>
+        <cylinder radius="${0.2 - center * 0.05}" length="0.05" />
       </geometry>
-	<origin rpy="3.1355 -1.3045 0.0025" xyz="0.3158 -0.0021 0.51"/>
-    </visual>
-  </link>
-  <link name="laser_vert_top_right">
-    <visual>
-      <geometry>
-        <box size="0.062 0.062 0.087"/>
-      </geometry>
-	<origin rpy="-1.1760 0.6313 -1.9377" xyz="0.2978 -0.1450 1.8451"/>
+	<origin rpy="-1.57079 0 0" xyz="${-0.1 +  0.2 * center} ${reflect * 0.2} ${-0.025 * center}"/>
     </visual>
     <collision>
       <geometry>
-        <box size="0.062 0.062 0.087"/>
+      	<cylinder radius="${0.2 - center * 0.05}" length="0.05" />
       </geometry>
-	<origin rpy="-1.1760 0.6313 -1.9377" xyz="0.2978 -0.1450 1.8451"/>
+			<origin rpy="-1.57079 0 0" xyz="${-0.1 +  0.2 * center} ${reflect * 0.2} ${-0.025 * center}"/>
     </collision>
   </link>
-  <link name="laser_vert_top_left">
-    <visual>
-      <geometry>
-        <box size="0.062 0.062 0.087"/>
-      </geometry>
-	<origin rpy="1.1780 0.6198 1.9560" xyz="0.2997 0.1531 1.8443"/>
-    </visual>
-    <collision>
-      <geometry>
-        <box size="0.062 0.062 0.087"/>
-      </geometry>
-	<origin rpy="1.1780 0.6198 1.9560" xyz="0.2997 0.1531 1.8443"/>
-    </collision>
-  </link>
-  <link name="laser_horiz">
-    <visual>
-      <geometry>
-        <cylinder length="0.072" radius="0.052"/>
-      </geometry>
-	<origin rpy="-0.0012068 0.114646 -0.0015308" xyz="0.2325 0.0001 1.9201"/>
-    </visual>
-    <collision>
-      <geometry>
-        <cylinder length="0.072" radius="0.052"/>
-      </geometry>
-	<origin rpy="-0.0012068 0.114646 -0.0015308" xyz="0.2325 0.0001 1.9201"/>
-    </collision>
-  </link>
-  <xacro:macro name="xacro_name" params="suffix reflect">
-  <link name="wheel_${suffix}">
-    <visual>
-      <geometry>
-        <cylinder length="0.05" radius="0.2"/>
-      </geometry>
-	<origin rpy="-1.57079 0 0" xyz="-0.1 0.4 0"/>
-    </visual>
-    <collision>
-      <geometry>
-        <cylinder length="0.05" radius="0.2"/>
-      </geometry>
-	<origin rpy="-1.57079 0 0" xyz="-0.1 0.4 0"/>
-    </collision>
-  </link>
-  <joint name="base_wheel_${suffix}_joint" type="fixed">
+  <joint name="base_wheel_${suffix}_joint" type="continuous">
 	<parent link="base"/>
 	<child link="wheel_${suffix}"/>
-	<origin xyz="-0.1 0.4 0"/>
+	<origin xyz="${-0.1 +  0.2 * center} ${reflect * 0.4} ${-0.025 * center}" rpy="0 -1.57079 0"/>
 	<limit velocity = "1" effort = "1"/>
   </joint>
   </xacro:macro>
-  <xacro:xacro_name suffix="left" reflect="1" />
-  <joint name="base_laser_vert_bottom_joint" type="fixed">
-    <parent link="base"/>
-    <child link="laser_vert_bottom"/>
-    <origin xyz="0.3158 -0.0021 0.5100"/>
-  </joint>
-  <joint name="base_laser_vert_top_right_joint" type="fixed">
-    <parent link="base"/>
-    <child link="laser_vert_top_right"/>
-    <origin xyz="0.2978 -0.1450 1.8451"/>
-  </joint>
-  <joint name="base_laser_vert_top_left_joint" type="fixed">
-    <parent link="base"/>
-    <child link="laser_vert_top_left"/>
-    <origin xyz="0.2997 0.1531 1.8443"/>
-  </joint>
-  <joint name="base_laser_horiz_joint" type="fixed">
-    <parent link="base"/>
-    <child link="laser_horiz"/>
-    <origin xyz="0.2325 0.0001 1.9201"/>
-  </joint>
+  <xacro:xacro_name suffix="left" reflect="1" center="0"/>
+	<xacro:xacro_name suffix="right" reflect="-1" center="0"/>
+	<xacro:xacro_name suffix="center" reflect="0" center="1"/>
 </robot>

Commit message: final commit

File: urdf/newrobot.urdf (robot description, URDF)
Before this commit: robot robot, 9 links, 8 joints
Joints:
- joint base_wheel_center_joint: axis (none) -> 0 1 0; origin xyz=0.1 0.0 -0.025 rpy=-1.57079 0 0 -> xyz=0.1 0.0 -0.025 rpy=0 -1.57079 0
- joint base_wheel_left_joint: axis (none) -> 0 1 0; origin xyz=-0.1 0.4 -0.0 rpy=-1.57079 0 0 -> xyz=-0.1 0.2 -0.0 rpy=0 -1.57079 0
- joint base_wheel_right_joint: axis (none) -> 0 1 0; origin xyz=-0.1 -0.4 -0.0 rpy=-1.57079 0 0 -> xyz=-0.1 -0.2 -0.0 rpy=0 -1.57079 0

File: urdf/torobot.xacro (robot description, xacro)
@@ -6,5 +6,5 @@
         <box size="0.94 0.78 1.98"/>
       </geometry>
-	<origin xyz="0 0 0.99"/>
+			<origin xyz="0 0 0.99"/>
     </visual>
     <collision>
@@ -39,12 +39,13 @@
       	<cylinder radius="${0.2 - center * 0.05}" length="0.05" />
       </geometry>
-			<origin rpy="-1.57079 0 0" xyz="${-0.1 +  0.2 * center} ${reflect * 0.2} ${-0.025 * center}"/>
+			<origin rpy="-1.57079 0 0" xyz="${-0.1 +  0.1 * center} ${reflect * 0.2} ${-0.025 * center}"/>
     </collision>
   </link>
   <joint name="base_wheel_${suffix}_joint" type="continuous">
-	<parent link="base"/>
-	<child link="wheel_${suffix}"/>
-	<origin xyz="${-0.1 +  0.2 * center} ${reflect * 0.4} ${-0.025 * center}" rpy="0 -1.57079 0"/>
-	<limit velocity = "1" effort = "1"/>
+		<axis xyz="0 1 0" />
+		<parent link="base"/>
+		<child link="wheel_${suffix}"/>
+		<origin xyz="${-0.1 +  0.2 * center} ${reflect * 0.2} ${-0.025 * center}" rpy="0 -1.57079 0"/>
+		<limit velocity = "1" effort = "1"/>
   </joint>
   </xacro:macro>
